File: kicad/split_3x_plate_bigger_encoder_gerber.kicad_pcb (KiCad board)
At the start: 2 copper layers, 122.2 x 121.2 mm, 6 parts

Commit message: added millmax hotswappable sockets
Other:
- net class Default removed
- net class Power removed
- net class TRRSData removed
